Commit message: Fix the bug in sick_s300.urdf.xacro file. The simulation only showed the data of ONE laserscan

File: urdf/sick_s300.urdf.xacro (robot description, xacro)
@@ -1,5 +1,5 @@
 <?xml version="1.0"?>
 <robot name="sensor_sick_s300" xmlns:xacro="http://www.ros.org/wiki/xacro">
-  <xacro:macro name="sensor_sick_s300" params="prefix parent prefix_topic:='front_laser' *origin">
+  <xacro:macro name="sensor_sick_s300" params="prefix parent *origin">
     <joint name="${prefix}_base_joint" type="fixed">
       <xacro:insert_block name="origin" />
@@ -9,5 +9,5 @@
 	<link name="${prefix}_base_link">
 		<collision>
-			<origin xyz="0 0 0" rpy="0 0 0"/>
+			<origin xyz="0 0 0.076" rpy="0 0 0"/>
 			<geometry>
 				<!--<box size="0.106 0.094 0.152"/>-->
@@ -64,5 +64,5 @@
 				</ray>
 				<plugin name="${prefix}_controller" filename="libgazebo_ros_laser.so">
-					<topicName>${prefix_topic}/scan</topicName>
+					<topicName>${prefix}/scan</topicName>
 					<frameName>/${prefix}_link</frameName><!-- if not global (leading /) sets the current namespace as a prefix (/ns/name_laser_link) -->
 				</plugin>
